Commit message: Added dynamic simplification

File: MeshSimplifier/example/pig/simple_pig/simple_pig3.obj.urdf (robot description, URDF)
Before this commit: robot pig.obj, 1 links, 0 joints
Links:
- link _name: geometry collision mesh filename=simple_pig3_vhacd.obj scale=1.0 1.0 1.0; visual mesh filename=simple_pig3.obj scale=1.0 1.0 1.0
